File: solarnode_medium/solarnode_medium.kicad_pcb (KiCad board)
At the start: 2 copper layers, 77 x 80 mm, 142 parts, among them J1 Conn_01x06, J2 Conn_01x04, Q1 AO3400, Q2 AO3400, Q3 AO3400, Q4 AO3400, Q5 Q_NPN_BEC, Q6 Q_NPN_BEC, Q7 Q_NPN_BEC, Q8 Q_NMOS_GSD, Q9 PMOS, SW1 SW_Push, SW2 SW_Push, SW3 SW_Push, U1 YX59012, U2 SGM2033-3.3, U3 MAX485E, U4 SGM48211, U5 SGM48211, U6 LM358, U7 YX59012, U8 CH32V203C8T6, U9 CN3058E, Y1 Crystal_GND24_Small, Y2 Crystal_Small

Commit message: 添加加速度传感器
Parts:
- added C39: 0.1uf, Capacitor_SMD:C_0402_1005Metric, B.Cu at (137.6, 118.6)
- added U10: QMA6100P, Package_LGA:LGA-12_2x2mm_P0.5mm, B.Cu at (137.7, 120.4)
Routing:
- net GND: track 312.6 -> 322.5 mm
- net +3.3V: track 73.2 -> 81.5 mm
- net /MCU and Commication/SDA: track 45.2 -> 51.9 mm
- net /MCU and Commication/SCL: track 44.1 -> 48.9 mm

Commit message: 添加断线报警器探测线接口
Parts:
- added J3: Conn_01x02, Connector_PinHeader_2.54mm:PinHeader_1x02_P2.54mm_Vertical, F.Cu at (98.4, 122.8)
Connections:
- U8 pad 31: unconnected-(U8-PA10-Pad31) -> /MCU and Commication/DET_LINE1
- U8 pad 32: unconnected-(U8-PA11-Pad32) -> /MCU and Commication/DET_LINE2
Routing:
- net /MCU and Commication/DET_LINE1: track 0.00 -> 20.9 mm, vias 0 -> 1
- net /MCU and Commication/DET_LINE2: track 0.00 -> 20.0 mm, vias 0 -> 1
